File: hardware/pcbs/radxa_hat/radxa_hat.kicad_sch (KiCad schematic)
At the start: 10 parts, among them J1 RADXA_HEADER, J2 Header_01x06, J3 Header_01x04, J4 Header_01x08, J5 Header_01x04

Commit message: hat_pcbs: more space under MTA100 connectors as per datasheet
Parts:
- J2: Purpose Pin2 INT -> RST; Purpose Pin3 RST -> INT
Changed lines of the file:
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@@
 			)
 		)
-		(property "Purpose Pin2" "INT"
-			(at 210.82 67.31 0)
+		(property "Purpose Pin2" "RST"
+			(at 210.82 69.85 0)
 			(do_not_autoplace yes)
 			(effects
@@
 			)
 		)
-		(property "Purpose Pin3" "RST"
-			(at 210.82 69.85 0)
+		(property "Purpose Pin3" "INT"
+			(at 210.82 67.31 0)
 			(do_not_autoplace yes)
 			(effects
