File: hardware/pcbs/audio_experiments/mv2_taa3040/balanced_transformer_input.kicad_sch (KiCad schematic)
At the start: 2 parts

Commit message: test pcb almost done
Connections:
- net COLD: now also D3.2 (I/O1); no longer D3.3 (I/O2)
- net HOT: now also D3.3 (I/O2); no longer D3.2 (I/O1)
Changed lines of the file:
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@@
 		(lib_id "Power_Protection:PRTR5V0U2X")
 		(at 181.61 91.44 270)
+		(mirror x)
 		(unit 1)
 		(exclude_from_sim no)
@@
 		(dnp no)
 		(property "Reference" "D3"
+			(at 185.42 100.33 90)
+			(effects
+				(font
+					(size 1.27 1.27)
+				)
+				(justify left)
+			)
+		)
+		(property "Value" "PRTR5V0U2X"
 			(at 185.42 82.55 90)
 			(effects
@@
 			)
 		)
-		(property "Value" "PRTR5V0U2X"
-			(at 185.42 100.33 90)
-			(effects
-				(font
-					(size 1.27 1.27)
-				)
-				(justify left)
-			)
-		)
 		(property "Footprint" "Package_TO_SOT_SMD:SOT-143"
-			(at 181.61 92.964 0)
+			(at 181.61 89.916 0)
 			(effects
 				(font
@@
 		)
 		(property "Datasheet" "https://assets.nexperia.com/documents/data-sheet/PRTR5V0U2X.pdf"
-			(at 181.61 92.964 0)
+			(at 181.61 89.916 0)
 			(effects
 				(font
