File: hardware/pcbs/audio_experiments/mv2_taa3040/conn_and_power.kicad_sch (KiCad schematic)
At the start: 5 parts, among them J4 Interconnect, U3 LP5907MFX-3.3

Commit message: finalise board
Parts:
- renumbered C29 to C30, C30 to C31
Changed lines of the file:
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@@
 		(on_board yes)
 		(dnp no)
-		(property "Reference" "#PWR065"
+		(property "Reference" "#PWR067"
 			(at 156.21 95.25 0)
 			(effects
@@
 			(project "mv2_taa3040"
 				(path "/41a55a1d-5108-482f-b313-9eaa5d011dff/cad1070f-df9f-433f-9c9e-3f26e05af870"
-					(reference "#PWR065")
+					(reference "#PWR067")
 					(unit 1)
 				)
@@
 		(on_board yes)
 		(dnp no)
-		(property "Reference" "#PWR060"
+		(property "Reference" "#PWR062"
 			(at 87.63 104.14 0)
 			(effects
@@
 			(project "mv2_taa3040"
 				(path "/41a55a1d-5108-482f-b313-9eaa5d011dff/cad1070f-df9f-433f-9c9e-3f26e05af870"
-					(reference "#PWR060")
+					(reference "#PWR062")
 					(unit 1)
 				)
@@
 		(on_board yes)
 		(dnp no)
-		(property "Reference" "#PWR063"
+		(property "Reference" "#PWR065"
 			(at 121.92 95.25 0)
 			(effects
@@
 			(project "mv2_taa3040"
 				(path "/41a55a1d-5108-482f-b313-9eaa5d011dff/cad1070f-df9f-433f-9c9e-3f26e05af870"
-					(reference "#PWR063")
+					(reference "#PWR065")
 					(unit 1)
 				)
@@
 		(dnp no)
 		(fields_autoplaced yes)
-		(property "Reference" "#PWR058"
+		(property "Reference" "#PWR060"
 			(at 77.47 86.36 0)
 			(effects
@@
 			(project "mv2_taa3040"
 				(path "/41a55a1d-5108-482f-b313-9eaa5d011dff/cad1070f-df9f-433f-9c9e-3f26e05af870"
-					(reference "#PWR058")
+					(reference "#PWR060")
 					(unit 1)
 				)
@@
 		(dnp no)
 		(fields_autoplaced yes)
-		(property "Reference" "#PWR061"
+		(property "Reference" "#PWR063"
 			(at 87.63 121.92 0)
 			(effects
@@
 			(project "mv2_taa3040"
 				(path "/41a55a1d-5108-482f-b313-9eaa5d011dff/cad1070f-df9f-433f-9c9e-3f26e05af870"
-					(reference "#PWR061")
+					(reference "#PWR063")
 					(unit 1)
 				)
@@
 		(on_board yes)
 		(dnp no)
-		(property "Reference" "#PWR067"
+		(property "Reference" "#PWR069"
 			(at 163.83 76.2 0)
 			(effects
@@
 			(project "mv2_taa3040"
 				(path "/41a55a1d-5108-482f-b313-9eaa5d011dff/cad1070f-df9f-433f-9c9e-3f26e05af870"
-					(reference "#PWR067")
+					(reference "#PWR069")
 					(unit 1)
 				)
@@
 		(dnp no)
 		(fields_autoplaced yes)
-		(property "Reference" "#PWR057"
+		(property "Reference" "#PWR059"
 			(at 77.47 76.2 0)
 			(effects
@@
 			(project ""
 				(path "/41a55a1d-5108-482f-b313-9eaa5d011dff/cad1070f-df9f-433f-9c9e-3f26e05af870"
-					(reference "#PWR057")
+					(reference "#PWR059")
 					(unit 1)
 				)
@@
 		(on_board yes)
 		(dnp no)
-		(property "Reference" "C29"
+		(property "Reference" "C30"
 			(at 121.92 80.01 0)
 			(effects
@@
 			(project "mv2_taa3040"
 				(path "/41a55a1d-5108-482f-b313-9eaa5d011dff/cad1070f-df9f-433f-9c9e-3f26e05af870"
-					(reference "C29")
+					(reference "C30")
 					(unit 1)
 				)
@@
 		(on_board yes)
 		(dnp no)
-		(property "Reference" "C30"
+		(property "Reference" "C31"
 			(at 156.21 80.01 0)
 			(effects
@@
 			(project "mv2_taa3040"
 				(path "/41a55a1d-5108-482f-b313-9eaa5d011dff/cad1070f-df9f-433f-9c9e-3f26e05af870"
-					(reference "C30")
+					(reference "C31")
 					(unit 1)
 				)
@@
 		(on_board yes)
 		(dnp no)
-		(property "Reference" "#PWR062"
+		(property "Reference" "#PWR064"
 			(at 121.92 76.2 0)
 			(effects
@@
 			(project "mv2_taa3040"
 				(path "/41a55a1d-5108-482f-b313-9eaa5d011dff/cad1070f-df9f-433f-9c9e-3f26e05af870"
-					(reference "#PWR062")
+					(reference "#PWR064")
 					(unit 1)
 				)
@@
 		(dnp no)
 		(fields_autoplaced yes)
-		(property "Reference" "#PWR059"
+		(property "Reference" "#PWR061"
 			(at 87.63 88.9 0)
 			(effects
@@
 			(project "mv2_taa3040"
 				(path "/41a55a1d-5108-482f-b313-9eaa5d011dff/cad1070f-df9f-433f-9c9e-3f26e05af870"
-					(reference "#PWR059")
+					(reference "#PWR061")
 					(unit 1)
 				)
@@
 		(on_board yes)
 		(dnp no)
-		(property "Reference" "#PWR066"
+		(property "Reference" "#PWR068"
 			(at 165.1 95.25 0)
 			(effects
@@
 			(project "mv2_taa3040"
 				(path "/41a55a1d-5108-482f-b313-9eaa5d011dff/cad1070f-df9f-433f-9c9e-3f26e05af870"
-					(reference "#PWR066")
+					(reference "#PWR068")
 					(unit 1)
 				)
@@
 		(dnp no)
 		(fields_autoplaced yes)
-		(property "Reference" "#PWR064"
+		(property "Reference" "#PWR066"
 			(at 139.7 95.25 0)
 			(effects
@@
 			(project "mv2_taa3040"
 				(path "/41a55a1d-5108-482f-b313-9eaa5d011dff/cad1070f-df9f-433f-9c9e-3f26e05af870"
-					(reference "#PWR064")
+					(reference "#PWR066")
 					(unit 1)
 				)
@@
 		(dnp no)
 		(fields_autoplaced yes)
-		(property "Reference" "#PWR056"
+		(property "Reference" "#PWR058"
 			(at 77.47 73.66 0)
 			(effects
@@
 			(project "mv2_taa3040"
 				(path "/41a55a1d-5108-482f-b313-9eaa5d011dff/cad1070f-df9f-433f-9c9e-3f26e05af870"
-					(reference "#PWR056")
-					(unit 1)
-				)
+					(reference "#PWR058")
+					(unit 1)
+				)

Commit message: update bom
Parts:
- J4: MPN Header_1x20 -> SSQ-120-03-T-S
Changed lines of the file:
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@@
 			)
 		)
-		(property "MPN" "Header_1x20"
+		(property "MPN" "SSQ-120-03-T-S"
 			(at 68.58 96.52 0)
 			(effects
