File: hardware/pcbs/audio_experiments/mv2_taa3040/input_frontend.kicad_sch (KiCad schematic)
At the start: 18 parts, among them J1 MTA100-3, Q1 2N7002, Q2 SI2309CDS-T1-GE3

Commit message: test pcb almost done
Parts:
- J1: Purpose Audio IN -> IN
Changed lines of the file:
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@@
 			)
 		)
-		(property "Purpose" "Audio IN"
+		(property "Purpose" "IN"
 			(at 96.52 125.73 0)
 			(effects

Commit message: finalise board
Parts:
- renumbered C20 to C21, C21 to C22, C22 to C23

Commit message: update bom
Parts:
- L1, L2: now in the parts list
Changed lines of the file:
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@@
 		(unit 1)
 		(exclude_from_sim no)
-		(in_bom no)
+		(in_bom yes)
 		(on_board yes)
 		(dnp no)
@@
 		(unit 1)
 		(exclude_from_sim no)
-		(in_bom no)
+		(in_bom yes)
 		(on_board yes)
 		(dnp no)
