File: hardware/pcbs/audio_experiments/mv2_taa3040/mv2_taa3040.kicad_sch (KiCad schematic)
At the start: 23 parts, among them U1 TCA9534, U2 TAA3040

Commit message: finalise board
Parts:
- added C1: 1μF, Capacitor_SMD:C_0805_2012Metric, symbol Device:C_Small
- renumbered C9 to C10, C1 to C2, C2 to C3, C3 to C4, C4 to C5, C5 to C6, C6 to C7, C7 to C8, C8 to C9
Connections:
- net +3.3V: now also C1.1
- net GND: now also C1.2

Commit message: update bom
Parts:
- JP1, JP2, JP3, JP4: now left out of the parts list
Changed lines of the file:
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@@
 		(unit 1)
 		(exclude_from_sim no)
-		(in_bom yes)
+		(in_bom no)
 		(on_board yes)
 		(dnp no)
@@
 		(unit 1)
 		(exclude_from_sim no)
-		(in_bom yes)
+		(in_bom no)
 		(on_board yes)
 		(dnp no)
@@
 		(unit 1)
 		(exclude_from_sim no)
-		(in_bom yes)
+		(in_bom no)
 		(on_board yes)
 		(dnp no)
@@
 		(unit 1)
 		(exclude_from_sim no)
-		(in_bom yes)
+		(in_bom no)
 		(on_board yes)
 		(dnp no)
