File: hardware/pcbs/audio_board/power.kicad_sch (KiCad schematic)
At the start: 27 parts, among them Q7 S8050, U5 LP5907MFX-3.3, U6 LM5158

Commit message: fix libraries
Parts:
- removed U6: LM5158, Package_DFN_QFN:WQFN-16-1EP_3x3mm_P0.5mm_EP1.68x1.68mm_ThermalVias, symbol Library:LM5158
- added U3: LM5158, symbol ics:LM5158
- renumbered C29 to C1, C50 to C10, C51 to C11, C52 to C12, C30 to C2, C37 to C3, C38 to C4, C39 to C5, C40 to C6, C47 to C7, C48 to C8, C49 to C9, D4 to D1, D5 to D2, D6 to D3, L7 to L1, L8 to L2, L9 to L3, Q7 to Q1, R48 to R10, R49 to R11, R50 to R12, R51 to R13, R52 to R14, R47 to R9, U5 to U2
Connections:
- net +5V: now also U3.3 (BIAS), U3.6 (EN)
- net GND: now also U3.1 (PGND), U3.16 (PGND), U3.7 (AGND)
- net SW: now also U3.13 (SW), U3.14 (SW)
- net at R10.2: now also U3.5 (RT)
- net at R11.2: now also U3.11 (MODE)
- net at C11.1, R14.2: now also U3.8 (COMP)
- net at C8.1: now also U3.10 (SS)
- net at R12.1, R13.2: now also U3.9 (FB)
- net at C7.1: now also U3.2 (VCC)
- no-connect marks 0 -> 1
Other:
- moved on the sheet: C1, C10, C11, C12, C2, C3, C4, C5, C6, C7, C8, C9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

Commit message: final touches to libraries
Parts:
- U3: footprint (none) -> Package_DFN_QFN:WQFN-16-1EP_3x3mm_P0.5mm_EP1.68x1.68mm_ThermalVias
Connections:
- net GND: now also U3.17 (EP)
Changed lines of the file:
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@@
 	(paper "A4")
+	(junction
+		(at 179.07 102.87)
+		(diameter 0)
+		(color 0 0 0 0)
+	)
 	(junction
 		(at 144.78 62.23)
@@
 	)
 	(junction
-		(at 180.34 102.87)
-		(diameter 0)
-		(color 0 0 0 0)
-	)
-	(junction
 		(at 207.01 92.71)
 		(diameter 0)
@@
 	)
 	(junction
+		(at 180.34 102.87)
+		(diameter 0)
+		(color 0 0 0 0)
+	)
+	(junction
 		(at 261.62 62.23)
 		(diameter 0)
@@
 	)
 	(junction
+		(at 181.61 102.87)
+		(diameter 0)
+		(color 0 0 0 0)
+	)
+	(junction
 		(at 201.93 62.23)
 		(diameter 0)
@@
 	(wire
 		(pts
+			(xy 180.34 102.87) (xy 180.34 110.49)
+		)
+		(stroke
+			(width 0)
+			(type default)
+		)
+	)
+	(wire
+		(pts
 			(xy 157.48 101.6) (xy 157.48 110.49)
 		)
@@
 	(wire
 		(pts
+			(xy 176.53 102.87) (xy 176.53 101.6)
+		)
+		(stroke
+			(width 0)
+			(type default)
+		)
+	)
+	(wire
+		(pts
 			(xy 199.39 90.17) (xy 199.39 92.71)
 		)
@@
 	(wire
 		(pts
+			(xy 179.07 102.87) (xy 176.53 102.87)
+		)
+		(stroke
+			(width 0)
+			(type default)
+		)
+	)
+	(wire
+		(pts
 			(xy 69.85 83.82) (xy 69.85 82.55)
 		)
@@
 	(wire
 		(pts
+			(xy 181.61 102.87) (xy 180.34 102.87)
+		)
+		(stroke
+			(width 0)
+			(type default)
+		)
+	)
+	(wire
+		(pts
 			(xy 140.97 87.63) (xy 140.97 62.23)
 		)
@@
 	(wire
 		(pts
-			(xy 180.34 101.6) (xy 180.34 102.87)
-		)
-		(stroke
-			(width 0)
-			(type default)
-		)
-	)
-	(wire
-		(pts
 			(xy 57.15 107.95) (xy 59.69 107.95)
 		)
@@
 	(wire
 		(pts
-			(xy 177.8 102.87) (xy 180.34 102.87)
-		)
-		(stroke
-			(width 0)
-			(type default)
-		)
-	)
-	(wire
-		(pts
 			(xy 201.93 86.36) (xy 201.93 87.63)
 		)
@@
 	(wire
 		(pts
-			(xy 180.34 102.87) (xy 182.88 102.87)
+			(xy 184.15 101.6) (xy 184.15 102.87)
 		)
 		(stroke
@@
 	(wire
 		(pts
-			(xy 177.8 101.6) (xy 177.8 102.87)
+			(xy 184.15 102.87) (xy 181.61 102.87)
 		)
 		(stroke
@@
 	(wire
 		(pts
+			(xy 179.07 101.6) (xy 179.07 102.87)
+		)
+		(stroke
+			(width 0)
+			(type default)
+		)
+	)
+	(wire
+		(pts
 			(xy 144.78 62.23) (xy 154.94 62.23)
 		)
@@
 	(wire
 		(pts
-			(xy 180.34 102.87) (xy 180.34 110.49)
-		)
-		(stroke
-			(width 0)
-			(type default)
-		)
-	)
-	(wire
-		(pts
 			(xy 196.85 96.52) (xy 196.85 95.25)
 		)
@@
 	(wire
 		(pts
-			(xy 182.88 102.87) (xy 182.88 101.6)
+			(xy 181.61 101.6) (xy 181.61 102.87)
 		)
 		(stroke
@@
 		(pts
 			(xy 165.1 76.2) (xy 166.37 76.2)
+		)
+		(stroke
+			(width 0)
+			(type default)
+		)
+	)
+	(wire
+		(pts
+			(xy 180.34 102.87) (xy 179.07 102.87)
 		)
 		(stroke
@@
 			)
 		)
-		(property "Footprint" ""
+		(property "Footprint" "Package_DFN_QFN:WQFN-16-1EP_3x3mm_P0.5mm_EP1.68x1.68mm_ThermalVias"
 			(at 168.91 67.31 0)
 			(effects
@@
 		(pin "11"
 		)
+		(pin "17"
+		)
 		(instances

Commit message: add vias and mask to ic packages and route dac
Parts:
- U3: footprint Package_DFN_QFN:WQFN-16-1EP_3x3mm_P0.5mm_EP1.68x1.68mm_ThermalVias -> ics:WQFN-16-1EP_3x3mm_P0.5mm_EP1.68x1.68mm_ThermalVias
Changed lines of the file:
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@@
 			)
 		)
-		(property "Footprint" "Package_DFN_QFN:WQFN-16-1EP_3x3mm_P0.5mm_EP1.68x1.68mm_ThermalVias"
+		(property "Footprint" "ics:WQFN-16-1EP_3x3mm_P0.5mm_EP1.68x1.68mm_ThermalVias"
 			(at 168.91 67.31 0)
 			(effects

Commit message: some more routing
Parts:
- renumbered R9 to R10, R10 to R11, R11 to R12, R12 to R13, R13 to R14, R14 to R15

Commit message: route some more
Parts:
- added C9: 0.1uF, Capacitor_SMD:C_0805_2012Metric, symbol Device:C_Small
- C4: value 22uF -> 47uF; footprint Capacitor_SMD:C_0805_2012Metric -> Capacitor_THT:CP_Radial_D5.0mm_P2.00mm; LCSC C45783 -> (none)
- renumbered C9 to C10, C10 to C11, C11 to C12, C12 to C13
Connections:
- net +5V: now also C9.1
- net GND: now also C9.2
Other:
- moved on the sheet: C5, C6

Commit message: routing almost complete
Parts:
- added C5, C6: 1μF, Capacitor_SMD:C_0805_2012Metric, symbol Device:C_Small
- renumbered C8 to C10, C9 to C11, C10 to C12, C11 to C13, C12 to C14, C13 to C15, C5 to C7, C6 to C8, C7 to C9
Connections:
- net +3.3VA: now also C5.1, C6.1
- net GND: now also C5.2, C6.2
Other:
- moved on the sheet: C3, D2

Commit message: finish routing
Parts:
- renumbered R11 to R10, R12 to R11, R13 to R12, R14 to R13, R15 to R14, R10 to R9
Changed lines of the file:
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@@
 		(on_board yes)
 		(dnp no)
-		(property "Reference" "R11"
+		(property "Reference" "R10"
 			(at 147.828 97.1463 0)
 			(effects
@@
 			(project "audio_board"
 				(path "/54443f96-c7c5-4432-b890-45b14a1547a1/23b45e70-9f0d-43c3-ad82-81d9481de3a2"
-					(reference "R11")
+					(reference "R10")
 					(unit 1)
 				)
@@
 		(on_board yes)
 		(dnp no)
-		(property "Reference" "R12"
+		(property "Reference" "R11"
 			(at 198.628 99.6863 0)
 			(effects
@@
 			(project "audio_board"
 				(path "/54443f96-c7c5-4432-b890-45b14a1547a1/23b45e70-9f0d-43c3-ad82-81d9481de3a2"
-					(reference "R12")
+					(reference "R11")
 					(unit 1)
 				)
@@
 		(on_board yes)
 		(dnp no)
-		(property "Reference" "R15"
+		(property "Reference" "R14"
 			(at 208.788 98.4163 0)
 			(effects
@@
 			(project "audio_board"
 				(path "/54443f96-c7c5-4432-b890-45b14a1547a1/23b45e70-9f0d-43c3-ad82-81d9481de3a2"
-					(reference "R15")
+					(reference "R14")
 					(unit 1)
 				)
@@
 		(on_board yes)
 		(dnp no)
-		(property "Reference" "R14"
+		(property "Reference" "R13"
 			(at 203.708 81.9063 0)
 			(effects
@@
 			(project "audio_board"
 				(path "/54443f96-c7c5-4432-b890-45b14a1547a1/23b45e70-9f0d-43c3-ad82-81d9481de3a2"
-					(reference "R14")
+					(reference "R13")
 					(unit 1)
 				)
@@
 		(on_board yes)
 		(dnp no)
-		(property "Reference" "R13"
+		(property "Reference" "R12"
 			(at 203.708 71.7463 0)
 			(effects
@@
 			(project "audio_board"
 				(path "/54443f96-c7c5-4432-b890-45b14a1547a1/23b45e70-9f0d-43c3-ad82-81d9481de3a2"
-					(reference "R13")
+					(reference "R12")
 					(unit 1)
 				)
@@
 		(dnp no)
 		(fields_autoplaced yes)
-		(property "Reference" "R10"
+		(property "Reference" "R9"
 			(at 62.23 67.3099 0)
 			(effects
@@
 			(project "audio_board"
 				(path "/54443f96-c7c5-4432-b890-45b14a1547a1/23b45e70-9f0d-43c3-ad82-81d9481de3a2"
-					(reference "R10")
-					(unit 1)
-				)
+					(reference "R9")
+					(unit 1)
+				)

Commit message: component values
Parts:
- C10: LCSC C1532 -> (none); MPN (none) -> C 22nF 16V 0805
- C11, C13, C8: value 0.1uF -> 100nF; LCSC C307331 -> (none); MPN (none) -> C 100nF 16V 0805
- C12: LCSC C21117 -> (none); MPN (none) -> C 33nF 16V 0805
- C14: LCSC C1664 -> (none); MPN (none) -> C 330pF 16V 0805
- C15: LCSC C1779 -> (none)
- C2: value 22uF -> 22μF; LCSC C45783 -> (none); MPN (none) -> C 22μF 16V 0805
- C4: value 47uF -> 47μF; MPN (none) -> C 47μF 16V P2
- C7: value 10uF -> 10μF; LCSC C15850 -> (none); MPN (none) -> C 10μF 16V 0805
- C9: value 1uF -> 1μF; LCSC C52923 -> (none); MPN (none) -> C 1μF 16V 0805
- D1: value B5819W SL -> Schottky; LCSC C8598 -> (none); MPN (none) -> B0540W
- D2: LCSC C478011 -> (none)
- D3: footprint Diode_SMD:D_SMA -> Diode_SMD:D_SMB; LCSC C14996 -> (none); MPN (none) -> SS210
- L1, L3: LCSC C1002 -> (none)
- Q1: LCSC C2146 -> (none)
- R10: LCSC C25768 -> (none)
- R11, R12: LCSC C25741 -> (none)
- R13: LCSC C25879 -> (none)
- R14: LCSC C25867 -> (none)
- R9: LCSC C25123 -> (none)
- U2: LCSC C80670 -> (none)
Changed lines of the file:
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@@
 			)
 		)
-		(property "LCSC" "C478011"
-			(at 80.01 114.3 90)
-			(effects
-				(font
-					(size 1.27 1.27)
-				)
-				(hide yes)
-			)
-		)
 		(pin "2"
 		)
@@
 			)
 		)
-		(property "LCSC" "C21117"
+		(property "MPN" "C 33nF 16V 0805"
 			(at 207.01 106.68 0)
 			(effects
@@
 			)
 		)
-		(property "LCSC" "C80670"
-			(at 67.31 110.49 0)
-			(effects
-				(font
-					(size 1.27 1.27)
-				)
-				(hide yes)
-			)
-		)
 		(pin "4"
 		)
@@
 			)
 		)
-		(property "Value" "47uF"
+		(property "Value" "47μF"
 			(at 95.25 74.0409 0)
 			(effects
@@
 			)
 		)
+		(property "MPN" "C 47μF 16V P2"
+			(at 91.44 73.66 0)
+			(effects
+				(font
+					(size 1.27 1.27)
+				)
+				(hide yes)
+			)
+		)
 		(pin "1"
 		)
@@
 			)
 		)
-		(property "Value" "B5819W SL"
+		(property "Value" "Schottky"
 			(at 81.28 70.1674 90)
 			(effects
@@
 			)
 		)
-		(property "LCSC" "C8598"
+		(property "MPN" "B0540W"
 			(at 78.74 68.58 90)
 			(effects
@@
 			)
 		)
-		(property "LCSC" "C1002"
-			(at 54.61 63.5 90)
-			(effects
-				(font
-					(size 1.27 1.27)
-				)
-				(hide yes)
-			)
-		)
 		(pin "1"
 		)
@@
 			)
 		)
-		(property "Value" "0.1uF"
+		(property "Value" "100nF"
 			(at 216.9541 69.8636 0)
 			(effects
@@
 			)
 		)
-		(property "LCSC" "C307331"
+		(property "MPN" "C 100nF 16V 0805"
 			(at 214.63 68.58 0)
 			(effects
@@
 			)
 		)
-		(property "LCSC" "C25768"
-			(at 146.05 97.79 0)
-			(effects
-				(font
-					(size 1.27 1.27)
-				)
-				(hide yes)
-			)
-		)
 		(pin "1"
 		)
@@
 			)
 		)
-		(property "LCSC" "C1002"
-			(at 231.14 62.23 90)
-			(effects
-				(font
-					(size 1.27 1.27)
-				)
-				(hide yes)
-			)
-		)
 		(pin "1"
 		)
@@
 			)
 		)
-		(property "Value" "10uF"
+		(property "Value" "10μF"
 			(at 140.97 68.5862 0)
 			(effects
@@
 			)
 		)
-		(property "LCSC" "C15850"
+		(property "MPN" "C 10μF 16V 0805"
 			(at 138.43 67.31 0)
 			(effects
@@
 			)
 		)
-		(property "Value" "0.1uF"
+		(property "Value" "100nF"
 			(at 150.9141 68.5936 0)
 			(effects
@@
 			)
 		)
-		(property "LCSC" "C307331"
+		(property "MPN" "C 100nF 16V 0805"
 			(at 148.59 67.31 0)
 			(effects
@@
 			)
 		)
-		(property "LCSC" "C25741"
-			(at 196.85 100.33 0)
-			(effects
-				(font
-					(size 1.27 1.27)
-				)
-				(hide yes)
-			)
-		)
 		(pin "1"
 		)
@@
 			)
 		)
-		(property "LCSC" "C25867"
-			(at 207.01 99.06 0)
-			(effects
-				(font
-					(size 1.27 1.27)
-				)
-				(hide yes)
-			)
-		)
 		(pin "1"
 		)
@@
 			)
 		)
-		(property "LCSC" "C1532"
-			(at 157.48 99.06 0)
+		(property "ESR" "38mohm"
+			(at 164.338 102.616 0)
 			(effects
 				(font
 					(size 1.27 1.27)
 				)
-				(hide yes)
 			)
 		)
-		(property "ESR" "38mohm"
-			(at 164.338 102.616 0)
+		(property "MPN" "C 22nF 16V 0805"
+			(at 157.48 99.06 0)
 			(effects
 				(font
 					(size 1.27 1.27)
 				)
+				(hide yes)
 			)
 		)
@@
 			)
 		)
-		(property "LCSC" "C25879"
-			(at 201.93 82.55 0)
-			(effects
-				(font
-					(size 1.27 1.27)
-				)
-				(hide yes)
-			)
-		)
 		(pin "1"
 		)
@@
 			)
 		)
-		(property "Value" "1uF"
+		(property "Value" "1μF"
 			(at 157.48 81.2862 0)
 			(effects
@@
 			)
 		)
-		(property "LCSC" "C52923 "
+		(property "MPN" "C 1μF 16V 0805"
 			(at 154.94 80.01 0)
 			(effects
@@
 			)
 		)
-		(property "Footprint" "Diode_SMD:D_SMA"
+		(property "Footprint" "Diode_SMD:D_SMB"
 			(at 194.31 62.23 0)
 			(effects
@@
 			)
 		)
-		(property "LCSC" "C14996"
-			(at 194.31 62.23 90)
+		(property "MPN" "SS210"
+			(at 194.31 62.23 0)
 			(effects
 				(font
@@
 			)
 		)
-		(property "LCSC" "C1779"
-			(at 226.06 68.58 0)
-			(effects
-				(font
-					(size 1.27 1.27)
-				)
-				(hide yes)
-			)
-		)
 		(property "DatasheetRef" "C5"
 			(at 226.06 68.58 0)
@@
 			)
 		)
-		(property "LCSC" "C25741"
-			(at 201.93 72.39 0)
-			(effects
-				(font
-					(size 1.27 1.27)
-				)
-				(hide yes)
-			)
-		)
 		(pin "1"
 		)
@@
 			)
 		)
-		(property "LCSC" "C2146"
-			(at 69.85 66.04 90)
-			(effects
-				(font
-					(size 1.27 1.27)
-				)
-				(hide yes)
-			)
-		)
 		(pin "2"
 		)
@@
 			)
 		)
-		(property "Value" "22uF"
+		(property "Value" "22μF"
 			(at 71.12 82.55 0)
 			(effects
@@
 			)
 		)
-		(property "LCSC" "C45783"
+		(property "MPN" "C 22μF 16V 0805"
 			(at 69.85 78.74 0)
 			(effects
@@
 			)
 		)
-		(property "Value" "0.1uF"
+		(property "Value" "100nF"
 			(at 161.0741 68.5936 0)
 			(effects
@@
 			)
 		)
-		(property "LCSC" "C307331"
+		(property "MPN" "C 100nF 16V 0805"
 			(at 158.75 67.31 0)
 			(effects
@@
 			)
 		)
-		(property "LCSC" "C25123"
-			(at 59.69 68.58 0)
-			(effects
-				(font
-					(size 1.27 1.27)
-				)
-				(hide yes)
-			)
-		)
 		(pin "1"
 		)
@@
 			)
 		)
-		(property "LCSC" "C1664"
+		(property "MPN" "C 330pF 16V 0805"
 			(at 217.17 99.06 0)
 			(effects
