File: hardware/pcbs/audio_board/adc.kicad_sch (KiCad schematic)
At the start: 10 parts, among them U3 TAA3040

Commit message: fix libraries
Parts:
- removed U3: TAA3040, Package_DFN_QFN:WQFN-24-1EP_4x4mm_P0.5mm_EP2.6x2.6mm, symbol Library:TAA3040
- added U6: TAA3040, Package_DFN_QFN:WQFN-24-1EP_4x4mm_P0.5mm_EP2.6x2.6mm, symbol audio_ics:TAA3040
- renumbered C53 to C27, C15 to C28, C16 to C29, C17 to C30, C18 to C31, C19 to C32, C20 to C33, C21 to C34, C22 to C35
Connections:
- net +3.3V: now also U6.14 (~{SHDNZ}), U6.15 (ADDR1), U6.19 (IOVDD)
- net +3.3VA: now also U6.1 (AVDD)
- net BCLK: now also U6.22 (BCLK)
- net DOUT: now also U6.21 (SDOUT)
- net FSYNC: now also U6.23 (FSYNC)
- net GND: now also U6.16 (ADDR0), U6.25 (VSS), U6.4 (AVSS)
- net IN1+: now also U6.6 (IN1+)
- net IN1-: now also U6.7 (IN1-)
- net IN2+: now also U6.8 (IN2+)
- net IN2-: now also U6.9 (IN2-)
- net IN3+: now also U6.10 (IN3+)
- net IN3-: now also U6.11 (IN3-)
- net IN4+: now also U6.12 (IN4+)
- net IN4-: now also U6.13 (IN4-)
- net SCL: now also U6.17 (SCL)
- net SDA: now also U6.18 (SDA)
- net at C27.1: now also U6.3 (VREF)
- net at C34.1, C35.1: now also U6.24 (DREG)
- net at C28.1, C29.1: now also U6.2 (AREG)
Other:
- moved on the sheet: C30, C31, C32, C33

Commit message: add vias and mask to ic packages and route dac
Parts:
- U6: footprint Package_DFN_QFN:WQFN-24-1EP_4x4mm_P0.5mm_EP2.6x2.6mm -> ics:WQFN-24-1EP_4x4mm_P0.5mm_EP2.6x2.6mm
Changed lines of the file:
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@@
 			)
 		)
-		(property "Footprint" "Package_DFN_QFN:WQFN-24-1EP_4x4mm_P0.5mm_EP2.6x2.6mm"
+		(property "Footprint" "ics:WQFN-24-1EP_4x4mm_P0.5mm_EP2.6x2.6mm"
 			(at 151.13 62.23 0)
 			(effects

Commit message: route some more
Parts:
- renumbered C27 to C28, C28 to C29, C29 to C30, C30 to C31, C31 to C32, C32 to C33, C33 to C34, C34 to C35, C35 to C36
Changed lines of the file:
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@@
 		(dnp no)
 		(fields_autoplaced yes)
-		(property "Reference" "C27"
+		(property "Reference" "C28"
 			(at 93.98 77.4762 0)
 			(effects
@@
 			(project "audio_board"
 				(path "/54443f96-c7c5-4432-b890-45b14a1547a1/f61319fa-7c7c-4923-baf7-ddc2208dd523"
-					(reference "C27")
+					(reference "C28")
 					(unit 1)
 				)
@@
 		(dnp no)
 		(fields_autoplaced yes)
-		(property "Reference" "C31"
+		(property "Reference" "C32"
 			(at 135.89 54.6162 0)
 			(effects
@@
 			(project "audio_board"
 				(path "/54443f96-c7c5-4432-b890-45b14a1547a1/f61319fa-7c7c-4923-baf7-ddc2208dd523"
-					(reference "C31")
+					(reference "C32")
 					(unit 1)
 				)
@@
 		(dnp no)
 		(fields_autoplaced yes)
-		(property "Reference" "C32"
+		(property "Reference" "C33"
 			(at 157.48 54.6162 0)
 			(effects
@@
 			(project "audio_board"
 				(path "/54443f96-c7c5-4432-b890-45b14a1547a1/f61319fa-7c7c-4923-baf7-ddc2208dd523"
-					(reference "C32")
+					(reference "C33")
 					(unit 1)
 				)
@@
 		(dnp no)
 		(fields_autoplaced yes)
-		(property "Reference" "C30"
+		(property "Reference" "C31"
 			(at 127 54.6162 0)
 			(effects
@@
 			(project "audio_board"
 				(path "/54443f96-c7c5-4432-b890-45b14a1547a1/f61319fa-7c7c-4923-baf7-ddc2208dd523"
-					(reference "C30")
+					(reference "C31")
 					(unit 1)
 				)
@@
 		(dnp no)
 		(fields_autoplaced yes)
-		(property "Reference" "C35"
+		(property "Reference" "C36"
 			(at 186.69 66.0462 0)
 			(effects
@@
 			(project "audio_board"
 				(path "/54443f96-c7c5-4432-b890-45b14a1547a1/f61319fa-7c7c-4923-baf7-ddc2208dd523"
-					(reference "C35")
+					(reference "C36")
 					(unit 1)
 				)
@@
 		(dnp no)
 		(fields_autoplaced yes)
-		(property "Reference" "C28"
+		(property "Reference" "C29"
 			(at 104.14 66.0462 0)
 			(effects
@@
 			(project "audio_board"
 				(path "/54443f96-c7c5-4432-b890-45b14a1547a1/f61319fa-7c7c-4923-baf7-ddc2208dd523"
-					(reference "C28")
+					(reference "C29")
 					(unit 1)
 				)
@@
 		(dnp no)
 		(fields_autoplaced yes)
-		(property "Reference" "C33"
+		(property "Reference" "C34"
 			(at 167.64 54.6162 0)
 			(effects
@@
 			(project "audio_board"
 				(path "/54443f96-c7c5-4432-b890-45b14a1547a1/f61319fa-7c7c-4923-baf7-ddc2208dd523"
-					(reference "C33")
+					(reference "C34")
 					(unit 1)
 				)
@@
 		(dnp no)
 		(fields_autoplaced yes)
-		(property "Reference" "C29"
+		(property "Reference" "C30"
 			(at 113.03 66.0462 0)
 			(effects
@@
 			(project "audio_board"
 				(path "/54443f96-c7c5-4432-b890-45b14a1547a1/f61319fa-7c7c-4923-baf7-ddc2208dd523"
-					(reference "C29")
+					(reference "C30")
 					(unit 1)
 				)
@@
 		(dnp no)
 		(fields_autoplaced yes)
-		(property "Reference" "C34"
+		(property "Reference" "C35"
 			(at 176.53 66.0462 0)
 			(effects
@@
 			(project "audio_board"
 				(path "/54443f96-c7c5-4432-b890-45b14a1547a1/f61319fa-7c7c-4923-baf7-ddc2208dd523"
-					(reference "C34")
-					(unit 1)
-				)
+					(reference "C35")
+					(unit 1)
+				)

Commit message: routing almost complete
Parts:
- renumbered C28 to C30, C29 to C31, C30 to C32, C31 to C33, C32 to C34, C33 to C35, C34 to C36, C35 to C37, C36 to C38
Changed lines of the file:
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@@
 		(on_board yes)
 		(dnp no)
-		(property "Reference" "#PWR075"
+		(property "Reference" "#PWR077"
 			(at 133.35 66.04 0)
 			(effects
@@
 			(project "audio_board"
 				(path "/54443f96-c7c5-4432-b890-45b14a1547a1/f61319fa-7c7c-4923-baf7-ddc2208dd523"
-					(reference "#PWR075")
+					(reference "#PWR077")
 					(unit 1)
 				)
@@
 		(dnp no)
 		(fields_autoplaced yes)
-		(property "Reference" "C28"
+		(property "Reference" "C30"
 			(at 93.98 77.4762 0)
 			(effects
@@
 			(project "audio_board"
 				(path "/54443f96-c7c5-4432-b890-45b14a1547a1/f61319fa-7c7c-4923-baf7-ddc2208dd523"
-					(reference "C28")
+					(reference "C30")
 					(unit 1)
 				)
@@
 		(on_board yes)
 		(dnp no)
-		(property "Reference" "#PWR076"
+		(property "Reference" "#PWR078"
 			(at 142.24 52.07 0)
 			(effects
@@
 			(project "audio_board"
 				(path "/54443f96-c7c5-4432-b890-45b14a1547a1/f61319fa-7c7c-4923-baf7-ddc2208dd523"
-					(reference "#PWR076")
+					(reference "#PWR078")
 					(unit 1)
 				)
@@
 		(on_board yes)
 		(dnp no)
-		(property "Reference" "#PWR083"
+		(property "Reference" "#PWR085"
 			(at 166.37 109.22 0)
 			(effects
@@
 			(project "audio_board"
 				(path "/54443f96-c7c5-4432-b890-45b14a1547a1/f61319fa-7c7c-4923-baf7-ddc2208dd523"
-					(reference "#PWR083")
+					(reference "#PWR085")
 					(unit 1)
 				)
@@
 		(on_board yes)
 		(dnp no)
-		(property "Reference" "#PWR078"
+		(property "Reference" "#PWR080"
 			(at 151.13 52.07 0)
 			(effects
@@
 			(project "audio_board"
 				(path "/54443f96-c7c5-4432-b890-45b14a1547a1/f61319fa-7c7c-4923-baf7-ddc2208dd523"
-					(reference "#PWR078")
+					(reference "#PWR080")
 					(unit 1)
 				)
@@
 		(on_board yes)
 		(dnp no)
-		(property "Reference" "#PWR080"
+		(property "Reference" "#PWR082"
 			(at 154.94 66.04 0)
 			(effects
@@
 			(project "audio_board"
 				(path "/54443f96-c7c5-4432-b890-45b14a1547a1/f61319fa-7c7c-4923-baf7-ddc2208dd523"
-					(reference "#PWR080")
+					(reference "#PWR082")
 					(unit 1)
 				)
@@
 		(on_board yes)
 		(dnp no)
-		(property "Reference" "#PWR081"
+		(property "Reference" "#PWR083"
 			(at 165.1 66.04 0)
 			(effects
@@
 			(project "audio_board"
 				(path "/54443f96-c7c5-4432-b890-45b14a1547a1/f61319fa-7c7c-4923-baf7-ddc2208dd523"
-					(reference "#PWR081")
+					(reference "#PWR083")
 					(unit 1)
 				)
@@
 		(dnp no)
 		(fields_autoplaced yes)
-		(property "Reference" "C32"
+		(property "Reference" "C34"
 			(at 135.89 54.6162 0)
 			(effects
@@
 			(project "audio_board"
 				(path "/54443f96-c7c5-4432-b890-45b14a1547a1/f61319fa-7c7c-4923-baf7-ddc2208dd523"
-					(reference "C32")
+					(reference "C34")
 					(unit 1)
 				)
@@
 		(on_board yes)
 		(dnp no)
-		(property "Reference" "#PWR072"
+		(property "Reference" "#PWR074"
 			(at 101.6 77.47 0)
 			(effects
@@
 			(project "audio_board"
 				(path "/54443f96-c7c5-4432-b890-45b14a1547a1/f61319fa-7c7c-4923-baf7-ddc2208dd523"
-					(reference "#PWR072")
+					(reference "#PWR074")
 					(unit 1)
 				)
@@
 		(dnp no)
 		(fields_autoplaced yes)
-		(property "Reference" "C33"
+		(property "Reference" "C35"
 			(at 157.48 54.6162 0)
 			(effects
@@
 			(project "audio_board"
 				(path "/54443f96-c7c5-4432-b890-45b14a1547a1/f61319fa-7c7c-4923-baf7-ddc2208dd523"
-					(reference "C33")
+					(reference "C35")
 					(unit 1)
 				)
@@
 		(dnp no)
 		(fields_autoplaced yes)
-		(property "Reference" "C31"
+		(property "Reference" "C33"
 			(at 127 54.6162 0)
 			(effects
@@
 			(project "audio_board"
 				(path "/54443f96-c7c5-4432-b890-45b14a1547a1/f61319fa-7c7c-4923-baf7-ddc2208dd523"
-					(reference "C31")
+					(reference "C33")
 					(unit 1)
 				)
@@
 		(on_board yes)
 		(dnp no)
-		(property "Reference" "#PWR074"
+		(property "Reference" "#PWR076"
 			(at 124.46 66.04 0)
 			(effects
@@
 			(project "audio_board"
 				(path "/54443f96-c7c5-4432-b890-45b14a1547a1/f61319fa-7c7c-4923-baf7-ddc2208dd523"
-					(reference "#PWR074")
+					(reference "#PWR076")
 					(unit 1)
 				)
@@
 		(dnp no)
 		(fields_autoplaced yes)
-		(property "Reference" "C36"
+		(property "Reference" "C38"
 			(at 186.69 66.0462 0)
 			(effects
@@
 			(project "audio_board"
 				(path "/54443f96-c7c5-4432-b890-45b14a1547a1/f61319fa-7c7c-4923-baf7-ddc2208dd523"
-					(reference "C36")
+					(reference "C38")
 					(unit 1)
 				)
@@
 		(dnp no)
 		(fields_autoplaced yes)
-		(property "Reference" "#PWR077"
+		(property "Reference" "#PWR079"
 			(at 144.78 124.46 0)
 			(effects
@@
 			(project "audio_board"
 				(path "/54443f96-c7c5-4432-b890-45b14a1547a1/f61319fa-7c7c-4923-baf7-ddc2208dd523"
-					(reference "#PWR077")
+					(reference "#PWR079")
 					(unit 1)
 				)
@@
 		(on_board yes)
 		(dnp no)
-		(property "Reference" "#PWR071"
+		(property "Reference" "#PWR073"
 			(at 91.44 88.9 0)
 			(effects
@@
 			(project "audio_board"
 				(path "/54443f96-c7c5-4432-b890-45b14a1547a1/f61319fa-7c7c-4923-baf7-ddc2208dd523"
-					(reference "#PWR071")
+					(reference "#PWR073")
 					(unit 1)
 				)
@@
 		(on_board yes)
 		(dnp no)
-		(property "Reference" "#PWR073"
+		(property "Reference" "#PWR075"
 			(at 110.49 77.47 0)
 			(effects
@@
 			(project "audio_board"
 				(path "/54443f96-c7c5-4432-b890-45b14a1547a1/f61319fa-7c7c-4923-baf7-ddc2208dd523"
-					(reference "#PWR073")
+					(reference "#PWR075")
 					(unit 1)
 				)
@@
 		(on_board yes)
 		(dnp no)
-		(property "Reference" "#PWR084"
+		(property "Reference" "#PWR086"
 			(at 173.99 77.47 0)
 			(effects
@@
 			(project "audio_board"
 				(path "/54443f96-c7c5-4432-b890-45b14a1547a1/f61319fa-7c7c-4923-baf7-ddc2208dd523"
-					(reference "#PWR084")
+					(reference "#PWR086")
 					(unit 1)
 				)
@@
 		(dnp no)
 		(fields_autoplaced yes)
-		(property "Reference" "C29"
+		(property "Reference" "C31"
 			(at 104.14 66.0462 0)
 			(effects
@@
 			(project "audio_board"
 				(path "/54443f96-c7c5-4432-b890-45b14a1547a1/f61319fa-7c7c-4923-baf7-ddc2208dd523"
-					(reference "C29")
+					(reference "C31")
 					(unit 1)
 				)
@@
 		(dnp no)
 		(fields_autoplaced yes)
-		(property "Reference" "C34"
+		(property "Reference" "C36"
 			(at 167.64 54.6162 0)
 			(effects
@@
 			(project "audio_board"
 				(path "/54443f96-c7c5-4432-b890-45b14a1547a1/f61319fa-7c7c-4923-baf7-ddc2208dd523"
-					(reference "C34")
+					(reference "C36")
 					(unit 1)
 				)
@@
 		(dnp no)
 		(fields_autoplaced yes)
-		(property "Reference" "#PWR082"
+		(property "Reference" "#PWR084"
 			(at 176.53 100.33 0)
 			(effects
@@
 			(project "audio_board"
 				(path "/54443f96-c7c5-4432-b890-45b14a1547a1/f61319fa-7c7c-4923-baf7-ddc2208dd523"
-					(reference "#PWR082")
+					(reference "#PWR084")
 					(unit 1)
 				)
@@
 		(dnp no)
 		(fields_autoplaced yes)
-		(property "Reference" "#PWR079"
+		(property "Reference" "#PWR081"
 			(at 151.13 124.46 0)
 			(effects
@@
 			(project "audio_board"
 				(path "/54443f96-c7c5-4432-b890-45b14a1547a1/f61319fa-7c7c-4923-baf7-ddc2208dd523"
-					(reference "#PWR079")
+					(reference "#PWR081")
 					(unit 1)
 				)
@@
 		(on_board yes)
 		(dnp no)
-		(property "Reference" "#PWR085"
+		(property "Reference" "#PWR087"
 			(at 184.15 77.47 0)
 			(effects
@@
 			(project "audio_board"
 				(path "/54443f96-c7c5-4432-b890-45b14a1547a1/f61319fa-7c7c-4923-baf7-ddc2208dd523"
-					(reference "#PWR085")
+					(reference "#PWR087")
 					(unit 1)
 				)
@@
 		(dnp no)
 		(fields_autoplaced yes)
-		(property "Reference" "C30"
+		(property "Reference" "C32"
 			(at 113.03 66.0462 0)
 			(effects
@@
 			(project "audio_board"
 				(path "/54443f96-c7c5-4432-b890-45b14a1547a1/f61319fa-7c7c-4923-baf7-ddc2208dd523"
-					(reference "C30")
+					(reference "C32")
 					(unit 1)
 				)
@@
 		(dnp no)
 		(fields_autoplaced yes)
-		(property "Reference" "C35"
+		(property "Reference" "C37"
 			(at 176.53 66.0462 0)
 			(effects
@@
 			(project "audio_board"
 				(path "/54443f96-c7c5-4432-b890-45b14a1547a1/f61319fa-7c7c-4923-baf7-ddc2208dd523"
-					(reference "C35")
-					(unit 1)
-				)
+					(reference "C37")
+					(unit 1)
+				)

Commit message: component values
Parts:
- C30, C33, C36: value 1uF -> 1μF; MPN (none) -> C 1μF 16V 0805
- C31, C38: value 10uF -> 10μF; MPN (none) -> C 10μF 16V 0805
- C32, C34, C35, C37: MPN (none) -> C 100nF 16V 0805
Changed lines of the file:
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@@
 			)
 		)
-		(property "Value" "1uF"
+		(property "Value" "1μF"
 			(at 93.98 80.0162 0)
 			(effects
@@
 		)
 		(property "Description" "Unpolarized capacitor, small symbol"
+			(at 91.44 78.74 0)
+			(effects
+				(font
+					(size 1.27 1.27)
+				)
+				(hide yes)
+			)
+		)
+		(property "MPN" "C 1μF 16V 0805"
 			(at 91.44 78.74 0)
 			(effects
@@
 			)
 		)
+		(property "MPN" "C 100nF 16V 0805"
+			(at 133.35 55.88 0)
+			(effects
+				(font
+					(size 1.27 1.27)
+				)
+				(hide yes)
+			)
+		)
 		(pin "1"
 		)
@@
 			)
 		)
+		(property "MPN" "C 100nF 16V 0805"
+			(at 154.94 55.88 0)
+			(effects
+				(font
+					(size 1.27 1.27)
+				)
+				(hide yes)
+			)
+		)
 		(pin "1"
 		)
@@
 			)
 		)
-		(property "Value" "1uF"
+		(property "Value" "1μF"
 			(at 127 57.1562 0)
 			(effects
@@
 		)
 		(property "Description" "Unpolarized capacitor, small symbol"
+			(at 124.46 55.88 0)
+			(effects
+				(font
+					(size 1.27 1.27)
+				)
+				(hide yes)
+			)
+		)
+		(property "MPN" "C 1μF 16V 0805"
 			(at 124.46 55.88 0)
 			(effects
@@
 			)
 		)
-		(property "Value" "10uF"
+		(property "Value" "10μF"
 			(at 186.69 68.5862 0)
 			(effects
@@
 		)
 		(property "Description" "Unpolarized capacitor, small symbol"
+			(at 184.15 67.31 0)
+			(effects
+				(font
+					(size 1.27 1.27)
+				)
+				(hide yes)
+			)
+		)
+		(property "MPN" "C 10μF 16V 0805"
 			(at 184.15 67.31 0)
 			(effects
@@
 			)
 		)
-		(property "Value" "10uF"
+		(property "Value" "10μF"
 			(at 104.14 68.5862 0)
 			(effects
@@
 		)
 		(property "Description" "Unpolarized capacitor, small symbol"
+			(at 101.6 67.31 0)
+			(effects
+				(font
+					(size 1.27 1.27)
+				)
+				(hide yes)
+			)
+		)
+		(property "MPN" "C 10μF 16V 0805"
 			(at 101.6 67.31 0)
 			(effects
@@
 			)
 		)
-		(property "Value" "1uF"
+		(property "Value" "1μF"
 			(at 167.64 57.1562 0)
 			(effects
@@
 		)
 		(property "Description" "Unpolarized capacitor, small symbol"
+			(at 165.1 55.88 0)
+			(effects
+				(font
+					(size 1.27 1.27)
+				)
+				(hide yes)
+			)
+		)
+		(property "MPN" "C 1μF 16V 0805"
 			(at 165.1 55.88 0)
 			(effects
@@
 			)
 		)
+		(property "MPN" "C 100nF 16V 0805"
+			(at 110.49 67.31 0)
+			(effects
+				(font
+					(size 1.27 1.27)
+				)
+				(hide yes)
+			)
+		)
 		(pin "1"
 		)
@@
 			(at 173.99 67.31 0)
 			(effects
+				(font
+					(size 1.27 1.27)
+				)
+				(hide yes)
+			)
+		)
+		(property "MPN" "C 100nF 16V 0805"
+			(at 173.99 67.31 0)
+			(effects

Commit message: revise BOM
Parts:
- U6: MPN (none) -> TAA3040IRTWR
Changed lines of the file:
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@@
+			)
+		)
+		(property "MPN" "TAA3040IRTWR"
+			(at 151.13 62.23 0)
+			(effects
+				(font
+					(size 1.27 1.27)
+				)
+				(hide yes)
 			)
 		)
