File: hardware/pcbs/audio_board/dac.kicad_sch (KiCad schematic)
At the start: 9 parts, among them U4 TAD5242

Commit message: fix mistakes in audioboard design
Parts:
- removed R18: 4.7kΩ, Resistor_SMD:R_0805_2012Metric, symbol Device:R
Connections:
- net DOUT is gone; now on net GND: U4.4 (MD6)
- net GND: now also U4.13 (MD0)
Changed lines of the file:
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@@
 	(wire
 		(pts
-			(xy 106.68 129.54) (xy 106.68 125.73)
+			(xy 106.68 104.14) (xy 106.68 129.54)
 		)
 		(stroke
@@
 	(wire
 		(pts
+			(xy 165.1 119.38) (xy 165.1 129.54)
+		)
+		(stroke
+			(width 0)
+			(type default)
+		)
+	)
+	(wire
+		(pts
 			(xy 167.64 109.22) (xy 151.13 109.22)
 		)
@@
 		(pts
 			(xy 201.93 124.46) (xy 201.93 129.54)
-		)
-		(stroke
-			(width 0)
-			(type default)
-		)
-	)
-	(wire
-		(pts
-			(xy 106.68 118.11) (xy 106.68 104.14)
 		)
 		(stroke
@@
 		(shape input)
 		(at 165.1 78.74 180)
-		(effects
-			(font
-				(size 1.27 1.27)
-			)
-			(justify right)
-		)
-	)
-	(hierarchical_label "DOUT"
-		(shape output)
-		(at 165.1 119.38 180)
 		(effects
 			(font
@@
 	)
 	(symbol
-		(lib_id "Device:R")
-		(at 106.68 121.92 0)
+		(lib_id "power:GND")
+		(at 165.1 129.54 0)
 		(unit 1)
 		(exclude_from_sim no)
@@
 		(dnp no)
 		(fields_autoplaced yes)
-		(property "Reference" "R18"
-			(at 109.22 120.6499 0)
-			(effects
-				(font
-					(size 1.27 1.27)
-				)
-				(justify left)
-			)
-		)
-		(property "Value" "4.7kΩ"
-			(at 109.22 123.1899 0)
-			(effects
-				(font
-					(size 1.27 1.27)
-				)
-				(justify left)
-			)
-		)
-		(property "Footprint" "Resistor_SMD:R_0805_2012Metric"
-			(at 104.902 121.92 90)
-			(effects
-				(font
-					(size 1.27 1.27)
-				)
-				(hide yes)
-			)
-		)
-		(property "Datasheet" "~"
-			(at 106.68 121.92 0)
-			(effects
-				(font
-					(size 1.27 1.27)
-				)
-				(hide yes)
-			)
-		)
-		(property "Description" "Resistor"
-			(at 106.68 121.92 0)
-			(effects
-				(font
-					(size 1.27 1.27)
-				)
-				(hide yes)
-			)
-		)
-		(property "MPN" "R 4.7kΩ 125mW 1% 0805"
-			(at 106.68 121.92 0)
-			(effects
-				(font
-					(size 1.27 1.27)
-				)
-				(hide yes)
-			)
-		)
-		(pin "2"
+		(property "Reference" "#PWR0118"
+			(at 165.1 135.89 0)
+			(effects
+				(font
+					(size 1.27 1.27)
+				)
+				(hide yes)
+			)
+		)
+		(property "Value" "GND"
+			(at 165.1 134.62 0)
+			(effects
+				(font
+					(size 1.27 1.27)
+				)
+				(hide yes)
+			)
+		)
+		(property "Footprint" ""
+			(at 165.1 129.54 0)
+			(effects
+				(font
+					(size 1.27 1.27)
+				)
+				(hide yes)
+			)
+		)
+		(property "Datasheet" ""
+			(at 165.1 129.54 0)
+			(effects
+				(font
+					(size 1.27 1.27)
+				)
+				(hide yes)
+			)
+		)
+		(property "Description" "Power symbol creates a global label with name \"GND\" , ground"
+			(at 165.1 129.54 0)
+			(effects
+				(font
+					(size 1.27 1.27)
+				)
+				(hide yes)
+			)
 		)
 		(pin "1"
@@
 			(project "audio_board"
 				(path "/54443f96-c7c5-4432-b890-45b14a1547a1/c20e00b3-a078-47c9-844e-cc3fff4643af"
-					(reference "R19")
+					(reference "#PWR0119")
 					(unit 1)
 				)
 				(path "/54443f96-c7c5-4432-b890-45b14a1547a1/e4b4e226-c2a2-4edc-87fb-3e533fe789a5"
-					(reference "R18")
-					(unit 1)
-				)
+					(reference "#PWR0118")
+					(unit 1)
+				)
